File: boards/senior_design/senior_design.kicad_pcb (KiCad board)
At the start: 2 copper layers, 74.4 x 64.8 mm, 20 parts, among them J1 Main Board Connector, U11 UA741CP Op Amp, U3 AD620, U4 Balanced Demodulator, U7 UA741CP Op Amp

Commit message: merging local changes
Other:
- board text added: "Sensor Board Team 27"
Changed lines of the file:
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@@
   )
   (gr_rect (start 84.963 48.26) (end 159.385 113.03) (layer "Edge.Cuts") (width 0.1) (fill none))
+  (gr_text "Sensor Board\nTeam 27\n" (at 147.066 95.25) (layer "F.SilkS")
+    (effects (font (size 1 1) (thickness 0.15)))
+  )
   (segment (start 120.523 96.52) (end 120.523 93.472) (width 0.25) (layer "F.Cu") (net 2))
   (segment (start 120.142 89.948) (end 120.174 89.916) (width 0.25) (layer "F.Cu") (net 2))
