File: boards/microcontroller_board/microcontroller_board.kicad_pcb (KiCad board)
At the start: 2 copper layers, 99.1 x 95.2 mm, 21 parts, among them IC1 MAX038*, IC2 MAX038*, J1 Conn_01x03_Male, J2 Conn_01x03_Male, J3 Conn_01x03_Male, J4 Conn_01x03_Male, J5 Conn_01x04_Male, J6 Conn_01x04_Male, J7 Conn_02x11_Odd_Even, U1 ATmega328P-A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

Commit message: making sure I pushed everything
Parts:
- C1, C2, C3, C4: footprint Capacitor_SMD:C_0805_2012Metric_Pad1.18x1.45mm_HandSolder -> Capacitor_THT:C_Axial_L3.8mm_D2.6mm_P7.50mm_Horizontal
- R1, R2: footprint Resistor_SMD:R_0805_2012Metric_Pad1.20x1.40mm_HandSolder -> Resistor_THT:R_Axial_DIN0204_L3.6mm_D1.6mm_P1.90mm_Vertical
- moved C4 31.5 mm to (181.2, 110.0), turned to 90 degrees
- moved C3 24.4 mm to (176.8, 109.7)
- moved C1 4.50 mm to (102.2, 64.8), turned to 90 degrees
- moved R2 2.80 mm to (132.6, 72.9), turned to 90 degrees
- moved R1 1.02 mm to (101.3, 68.1), turned to -90 degrees
- moved C2 0.84 mm to (132.3, 65.2), turned to 90 degrees
Routing:
- net GND: track 48.6 -> 23.6 mm, vias 6 -> 4
- net Net-(C4-Pad1): track 27.8 -> 42.6 mm, vias 0 -> 2
- net Net-(C3-Pad2): track 16.3 -> 28.9 mm, vias 0 -> 2
- net Net-(C2-Pad2): track 5.06 -> 6.97 mm
- net Net-(C1-Pad2): track 7.49 -> 8.14 mm
