File: boards/microcontroller_board/microcontroller_board.kicad_sch (KiCad schematic)
At the start: 21 parts, among them IC1 MAX038*, IC2 MAX038*, J1 Conn_01x03_Male, J2 Conn_01x03_Male, J3 Conn_01x03_Male, J4 Conn_01x03_Male, J5 Conn_01x04_Male, J6 Conn_01x04_Male, J7 Conn_02x11_Odd_Even, U1 ATmega328P-A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

Commit message: making sure I pushed everything
Parts:
- added R3, R4, R5, R6: 1K, symbol Device:R
- added U2, U3: UA741CP, DIP794W45P254L959H508Q8, symbol uA741:UA741CP
- C1, C2, C3, C4: footprint Capacitor_SMD:C_0805_2012Metric_Pad1.18x1.45mm_HandSolder -> Capacitor_THT:C_Axial_L3.8mm_D2.6mm_P7.50mm_Horizontal
- R1, R2: footprint Resistor_SMD:R_0805_2012Metric_Pad1.20x1.40mm_HandSolder -> Resistor_THT:R_Axial_DIN0204_L3.6mm_D1.6mm_P1.90mm_Vertical
Connections:
- net +5V: now also U3.7 (VCC+)
- net GND: now also R3.2, R5.2
- new net: R3.1, R4.2, U2.2 (IN-)
- new net: R5.1, R6.2, U3.2 (IN-)
- new net: IC2.19 (OUT), U3.3 (IN+)
- new net: R6.1, U3.6 (OUT)
- new net: R4.1, U2.6 (OUT)
- new net: IC1.19 (OUT), U2.3 (IN+)
- now unconnected: J2.1 (Pin_1), J2.2 (Pin_2), J3.1 (Pin_1), J3.2 (Pin_2), J4.1 (Pin_1), J4.2 (Pin_2)
Other:
- note removed: "Power"
- moved on the sheet: J1
