File: boards/voltage_adder_board/voltage_adder_board/voltage_adder_board.kicad_sch (KiCad schematic)
At the start: 30 parts, among them J1 Conn_01x02_Female, J2 Conn_01x04, J3 Conn_01x02_Female, J4 Conn_01x02_Female, J5 Conn_01x03_Female, J6 Conn_01x03_Female, U1 UA741CP, U2 UA741CP, U3 UA741CP

Commit message: finished voltage adder board
Parts:
- added J7: Conn_01x03_Female, Connector_Molex:Molex_KK-254_AE-6410-03A_1x03_P2.54mm_Vertical, symbol Connector:Conn_01x03_Female
Connections:
- net +5V: now also J7.1 (Pin_1)
- net -5V: now also J7.2 (Pin_2)
- net GND: now also J7.3 (Pin_3)
Other:
- note added: "Power Connectors"
- note removed: "Power Connector"
Changed lines of the file:
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@@
+    (stroke (width 0) (type default) (color 0 0 0 0))
+  )
+  (wire (pts (xy 171.45 138.43) (xy 175.26 138.43))
     (stroke (width 0) (type default) (color 0 0 0 0))
   )
@@
     (effects (font (size 1.27 1.27)) (justify left bottom))
   )
-  (text "Power Connector" (at 162.56 151.13 0)
+  (text "Power Connectors\n" (at 158.75 128.27 0)
     (effects (font (size 1.27 1.27)) (justify left bottom))
   )
@@
     )
     (property "Datasheet" "~" (id 3) (at 143.51 50.8 0)
+      (effects (font (size 1.27 1.27)) hide)
+    )
+    (pin "1")
+    (pin "2")
+    (pin "3")
+  )
+  (symbol (lib_id "Connector:Conn_01x03_Female") (at 180.34 138.43 0) (unit 1)
+    (in_bom yes) (on_board yes)
+    (property "Reference" "J7" (id 0) (at 181.61 137.1599 0)
+      (effects (font (size 1.27 1.27)) (justify left))
+    )
+    (property "Value" "Conn_01x03_Female" (id 1) (at 166.37 148.59 0)
+      (effects (font (size 1.27 1.27)) (justify left))
+    )
+    (property "Footprint" "Connector_Molex:Molex_KK-254_AE-6410-03A_1x03_P2.54mm_Vertical" (id 2) (at 180.34 138.43 0)
+      (effects (font (size 1.27 1.27)) hide)
+    )
+    (property "Datasheet" "~" (id 3) (at 180.34 138.43 0)
       (effects (font (size 1.27 1.27)) hide)
     )
@@
     (pin "2")
   )
+  (symbol (lib_id "power:+5V") (at 175.26 135.89 0) (unit 1)
+    (in_bom yes) (on_board yes) (fields_autoplaced)
+    (property "Reference" "#PWR0121" (id 0) (at 175.26 139.7 0)
+      (effects (font (size 1.27 1.27)) hide)
+    )
+    (property "Value" "+5V" (id 1) (at 175.26 130.81 0))
+    (property "Footprint" "" (id 2) (at 175.26 135.89 0)
+      (effects (font (size 1.27 1.27)) hide)
+    )
+    (property "Datasheet" "" (id 3) (at 175.26 135.89 0)
+      (effects (font (size 1.27 1.27)) hide)
+    )
+    (pin "1")
+  )
   (symbol (lib_id "power:+5V") (at 153.67 135.89 0) (unit 1)
     (in_bom yes) (on_board yes) (fields_autoplaced)
@@
     (pin "2")
   )
+  (symbol (lib_id "power:-5V") (at 171.45 138.43 90) (unit 1)
+    (in_bom yes) (on_board yes)
+    (property "Reference" "#PWR0119" (id 0) (at 168.91 138.43 0)
+      (effects (font (size 1.27 1.27)) hide)
+    )
+    (property "Value" "-5V" (id 1) (at 170.18 142.24 0))
+    (property "Footprint" "" (id 2) (at 171.45 138.43 0)
+      (effects (font (size 1.27 1.27)) hide)
+    )
+    (property "Datasheet" "" (id 3) (at 171.45 138.43 0)
+      (effects (font (size 1.27 1.27)) hide)
+    )
+    (pin "1")
+  )
   (symbol (lib_id "power:GND") (at 73.66 142.24 270) (unit 1)
     (in_bom yes) (on_board yes)
@@
       (effects (font (size 1.27 1.27)) (justify left))
     )
-    (property "Value" "Conn_01x03_Female" (id 1) (at 160.02 139.6999 0)
+    (property "Value" "Conn_01x03_Female" (id 1) (at 143.51 148.59 0)
       (effects (font (size 1.27 1.27)) (justify left))
     )
@@
     (pin "2")
   )
+  (symbol (lib_id "power:GND") (at 175.26 140.97 0) (unit 1)
+    (in_bom yes) (on_board yes) (fields_autoplaced)
+    (property "Reference" "#PWR0120" (id 0) (at 175.26 147.32 0)
+      (effects (font (size 1.27 1.27)) hide)
+    )
+    (property "Value" "GND" (id 1) (at 175.26 146.05 0))
+    (property "Footprint" "" (id 2) (at 175.26 140.97 0)
+      (effects (font (size 1.27 1.27)) hide)
+    )
+    (property "Datasheet" "" (id 3) (at 175.26 140.97 0)
+      (effects (font (size 1.27 1.27)) hide)
+    )
+    (pin "1")
+  )
   (symbol (lib_id "Device:R") (at 190.5 68.58 90) (unit 1)
     (in_bom yes) (on_board yes) (fields_autoplaced)
@@
       (reference "#PWR0118") (unit 1) (value "-5V") (footprint "")
     )
+    (path "/8edd53b2-4877-4a5b-b217-9b3c553b9301"
+      (reference "#PWR0119") (unit 1) (value "-5V") (footprint "")
+    )
+    (path "/f90a51ff-416f-4eac-82ed-38c599a6ae3f"
+      (reference "#PWR0120") (unit 1) (value "GND") (footprint "")
+    )
+    (path "/48cffc50-fb06-4eb1-9b93-78f85a43b110"
+      (reference "#PWR0121") (unit 1) (value "+5V") (footprint "")
+    )
     (path "/be784310-ec98-4626-8958-169c17ee37d9"
       (reference "H1") (unit 1) (value "MountingHole") (footprint "MountingHole:MountingHole_3.2mm_M3")
@@
       (reference "J6") (unit 1) (value "Conn_01x03_Female") (footprint "Connector_Molex:Molex_KK-254_AE-6410-03A_1x03_P2.54mm_Vertical")
     )
+    (path "/1de9dde9-f32f-45ab-be8b-8ff4403cbd31"
+      (reference "J7") (unit 1) (value "Conn_01x03_Female") (footprint "Connector_Molex:Molex_KK-254_AE-6410-03A_1x03_P2.54mm_Vertical")
+    )
     (path "/5d22019e-730e-435b-bb8b-72e19a5bed0c"
